File: board/my_project.kicad_sch (KiCad schematic)
At the start: 3 parts, among them U1 LT1762

Commit message: added LCSC fields to components
Parts:
- R1: LCSC (none) -> 1234
- R2: LCSC (none) -> 4567
- U1: LCSC (none) -> 999
Changed lines of the file:
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@@
+			)
+		)
+		(property "LCSC" "4567"
+			(at 160.02 99.06 0)
+			(hide yes)
+			(show_name no)
+			(do_not_autoplace no)
+			(effects
+				(font
+					(size 1.27 1.27)
+				)
 			)
 		)
@@
 		)
 		(property "Description" "150mA, Adjustable, Low Noise, Micropower LDO Regulator, MSOP-8"
+			(at 135.89 95.25 0)
+			(hide yes)
+			(show_name no)
+			(do_not_autoplace no)
+			(effects
+				(font
+					(size 1.27 1.27)
+				)
+			)
+		)
+		(property "LCSC" "999"
 			(at 135.89 95.25 0)
 			(hide yes)
@@
 			(at 160.02 91.44 0)
 			(hide yes)
+			(show_name no)
+			(do_not_autoplace no)
+			(effects
+				(font
+					(size 1.27 1.27)
+				)
+			)
+		)
+		(property "LCSC" "1234"
+			(at 160.02 91.44 0)
+			(hide yes)
